File: grblPANEL_210x200_Front_Panel.kicad_pcb (KiCad board)
At the start: 2 copper layers, 200 x 210 mm, 0 parts

Commit message: Copper pours on front and back layers
Routing:
- added copper zone on B.Cu, net (none)
- added copper zone on F.Cu, net (none)
Other:
- board text removed: "<--- Move 2mm left for alignment? Or 2mm right to center between display bezel and edge?"
Changed lines of the file:
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@@
   )
   (net 0 "")
+  (gr_rect (start 55 40) (end 257 252)
+    (stroke (width 0.2) (type default)) (fill none) (layer "F.Cu"))
   (gr_line (start 140 176) (end 140 211)
     (stroke (width 0.25) (type default)) (layer "F.SilkS"))
@@
     )
   )
-  (gr_text "<--- Move 2mm left for alignment?\n       Or 2mm right to center between \n       display bezel and edge?" (at 242 89) (layer "User.1")
-    (effects (font (size 6 4) (thickness 0.15)) (justify left bottom))
+  (zone (net 0) (net_name "") (layers "F&B.Cu") (hatch edge 0.5)
+    (connect_pads (clearance 0.5))
+    (min_thickness 0.25) (filled_areas_thickness no)
+    (fill yes (thermal_gap 0.5) (thermal_bridge_width 0.5) (island_removal_mode 1) (island_area_min 10))
+    (polygon
+      (pts
+        (xy 55 40)
+        (xy 257 40)
+        (xy 257 252)
+        (xy 55 252)
+      )
+    )
   )
   (group "" (id d1fc8250-8049-47d1-a4d0-924568620361)
