File: grblPANEL_210x200_Front_Panel.kicad_pcb (KiCad board)
At the start: 2 copper layers, 200 x 210 mm, 0 parts

Commit message: Add info text to back of board
Parts:
- added G***: LOGO, dresco:OSHW_LOGO_10MM, B.Cu at (177.0, 54.5)
Other:
- board text added: "CC-BY-SA"
- board text added: "grblPANEL Rev B - 04/23 github.com/dresco/grblPANEL"
