File: grblPANEL_210x200_Front_Panel.kicad_pcb (KiCad board)
At the start: 2 copper layers, 200 x 210 mm, 1 part

Commit message: Add title block details
Other:
- board text added: "grblPANEL Rev A - 04/23 github.com/dresco/grblPANEL"
- board text removed: "grblPANEL Rev B - 04/23 github.com/dresco/grblPANEL"
Changed lines of the file:
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@@
   )
   (paper "A3")
+  (title_block
+    (title "grblPANEL - Front Panel")
+    (date "2023-04-28")
+    (rev "A")
+    (company "dresco")
+  )
   (layers
     (0 "F.Cu" signal)
@@
     (effects (font (size 3 2.5) (thickness 0.5) bold) (justify mirror))
   )
-  (gr_text "grblPANEL\nRev B - 04/23\ngithub.com/dresco/grblPANEL" (at 244 84 90) (layer "B.SilkS")
+  (gr_text "grblPANEL\nRev A - 04/23\ngithub.com/dresco/grblPANEL" (at 244 84 90) (layer "B.SilkS")
     (effects (font (size 3 2.5) (thickness 0.5) bold) (justify mirror))
   )
